File: Raspberry_modular_kicad/Raspberry_modular.kicad_sch (KiCad schematic)
At the start: 21 parts, among them J1 Raspberry_Pi_2_3, U1 MCP3008, U3 MCP3008

Commit message: [UDPT] All symbols are now in lib
Parts:
- H1, H2, H3, H4: symbol Mechanical:MountingHole -> Modular Shield:MountingHole
- J1: symbol Connector:Raspberry_Pi_2_3 -> Modular Shield:Raspberry_Pi_Header
- JP1: symbol Raspberry_modular-rescue:PINHD-1X6B-OhEye-eagle-import -> Modular Shield:PINHD-1X6B
- R4, R50, R51, R52, R53, R54, R55, R56: symbol Device:R -> Modular Shield:R
- U$3, U$5: symbol Raspberry_modular-rescue:PINHD-1X10-OhEye-eagle-import -> Modular Shield:PINHD-1X10
Changed lines of the file:
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@@
     (effects (font (size 1.27 1.27)) (justify right bottom))
   )
-  (symbol (lib_id "Raspberry_modular-rescue:PINHD-1X10-OhEye-eagle-import") (at 238.76 40.64 0) (unit 1)
+  (symbol (lib_id "Modular Shield:PINHD-1X10") (at 238.76 40.64 0) (unit 1)
     (in_bom yes) (on_board yes) (dnp no)
     (property "Reference" "U$3" (at 232.41 27.305 0)
@@
     )
   )
-  (symbol (lib_id "Mechanical:MountingHole") (at 128.27 27.94 0) (unit 1)
+  (symbol (lib_id "Modular Shield:MountingHole") (at 128.27 27.94 0) (unit 1)
     (in_bom yes) (on_board yes) (dnp no)
     (property "Reference" "H1" (at 130.81 26.7716 0)
@@
     )
   )
-  (symbol (lib_id "Mechanical:MountingHole") (at 128.27 33.02 0) (unit 1)
+  (symbol (lib_id "Modular Shield:MountingHole") (at 128.27 33.02 0) (unit 1)
     (in_bom yes) (on_board yes) (dnp no)
     (property "Reference" "H2" (at 130.81 31.8516 0)
@@
     )
   )
-  (symbol (lib_id "Mechanical:MountingHole") (at 128.27 38.1 0) (unit 1)
+  (symbol (lib_id "Modular Shield:MountingHole") (at 128.27 38.1 0) (unit 1)
     (in_bom yes) (on_board yes) (dnp no)
     (property "Reference" "H3" (at 130.81 36.9316 0)
@@
     )
   )
-  (symbol (lib_id "Mechanical:MountingHole") (at 128.27 43.18 0) (unit 1)
+  (symbol (lib_id "Modular Shield:MountingHole") (at 128.27 43.18 0) (unit 1)
     (in_bom yes) (on_board yes) (dnp no)
     (property "Reference" "H4" (at 130.81 42.0116 0)
@@
     )
   )
-  (symbol (lib_id "Device:R") (at 234.95 142.24 90) (unit 1)
+  (symbol (lib_id "Modular Shield:R") (at 234.95 142.24 90) (unit 1)
     (in_bom yes) (on_board yes) (dnp no)
     (property "Reference" "R4" (at 234.95 136.9822 90)
@@
     )
   )
-  (symbol (lib_id "Device:R") (at 234.95 147.32 90) (unit 1)
+  (symbol (lib_id "Modular Shield:R") (at 234.95 147.32 90) (unit 1)
     (in_bom yes) (on_board yes) (dnp no)
     (property "Reference" "R50" (at 234.95 142.0622 90)
@@
     )
   )
-  (symbol (lib_id "Device:R") (at 234.95 152.4 90) (unit 1)
+  (symbol (lib_id "Modular Shield:R") (at 234.95 152.4 90) (unit 1)
     (in_bom yes) (on_board yes) (dnp no)
     (property "Reference" "R51" (at 234.95 147.1422 90)
@@
     )
   )
-  (symbol (lib_id "Device:R") (at 234.95 157.48 90) (unit 1)
+  (symbol (lib_id "Modular Shield:R") (at 234.95 157.48 90) (unit 1)
     (in_bom yes) (on_board yes) (dnp no)
     (property "Reference" "R52" (at 234.95 152.2222 90)
@@
     )
   )
-  (symbol (lib_id "Device:R") (at 234.95 162.56 90) (unit 1)
+  (symbol (lib_id "Modular Shield:R") (at 234.95 162.56 90) (unit 1)
     (in_bom yes) (on_board yes) (dnp no)
     (property "Reference" "R53" (at 234.95 157.3022 90)
@@
     )
   )
-  (symbol (lib_id "Device:R") (at 234.95 167.64 90) (unit 1)
+  (symbol (lib_id "Modular Shield:R") (at 234.95 167.64 90) (unit 1)
     (in_bom yes) (on_board yes) (dnp no)
     (property "Reference" "R54" (at 234.95 162.3822 90)
@@
     )
   )
-  (symbol (lib_id "Device:R") (at 234.95 172.72 90) (unit 1)
+  (symbol (lib_id "Modular Shield:R") (at 234.95 172.72 90) (unit 1)
     (in_bom yes) (on_board yes) (dnp no)
     (property "Reference" "R55" (at 234.95 167.4622 90)
@@
     )
   )
-  (symbol (lib_id "Device:R") (at 234.95 177.8 90) (unit 1)
+  (symbol (lib_id "Modular Shield:R") (at 234.95 177.8 90) (unit 1)
     (in_bom yes) (on_board yes) (dnp no)
     (property "Reference" "R56" (at 234.95 172.5422 90)
@@
     )
   )
-  (symbol (lib_id "Connector:Raspberry_Pi_2_3") (at 49.53 78.74 0) (unit 1)
+  (symbol (lib_id "Modular Shield:Raspberry_Pi_Header") (at 49.53 78.74 0) (unit 1)
     (in_bom yes) (on_board yes) (dnp no)
     (property "Reference" "J1" (at 53.34 30.48 0)
@@
       (effects (font (size 1.27 1.27)) hide)
     )
-    (property "Datasheet" "https://www.raspberrypi.org/documentation/hardware/raspberrypi/schematics/rpi_SCH_3bplus_1p0_reduced.pdf" (at 49.53 78.74 0)
+    (property "Datasheet" "https://www.raspberrypi.org/documentation/hardware/raspberrypi/schematics/rpi_SCH_3bplus_1p0_reduced.pdf" (at 49.53 33.02 0)
       (effects (font (size 1.27 1.27)) hide)
     )
@@
     )
   )
-  (symbol (lib_id "Raspberry_modular-rescue:PINHD-1X10-OhEye-eagle-import") (at 269.24 40.64 0) (unit 1)
+  (symbol (lib_id "Modular Shield:PINHD-1X10") (at 269.24 40.64 0) (unit 1)
     (in_bom yes) (on_board yes) (dnp no)
     (property "Reference" "U$5" (at 262.89 27.305 0)
@@
     )
   )
-  (symbol (lib_id "Raspberry_modular-rescue:PINHD-1X6B-OhEye-eagle-import") (at 238.76 66.04 0) (unit 1)
+  (symbol (lib_id "Modular Shield:PINHD-1X6B") (at 238.76 66.04 0) (unit 1)
     (in_bom yes) (on_board yes) (dnp no)
     (property "Reference" "JP1" (at 232.41 55.245 0)

Commit message: [UDPT] Inputs on schematics
Other:
- note added: "Analog Input Regulators"
- moved on the sheet: U1, U3
