File: Raspberry_modular_kicad/Raspberry_modular.kicad_sch (KiCad schematic)
At the start: 21 parts, among them J1 Raspberry_Pi_2_3, U1 MCP3008, U3 MCP3008

Commit message: [UDPT] Inputs on schematics
Other:
- note added: "Analog Inputs Regulators"
- note added: "Digital Inputs Pull-Up"
- note removed: "Analog Input Regulators"
- moved on the sheet: R4, R50, R51, R52, R53, R54, R55, R56

Commit message: [UDPT] Shematics
Parts:
- JP5: value PINHD-1X8BIG -> PINHD-1X8; symbol Raspberry_modular-rescue:PINHD-1X8BIG-OhEye-eagle-import -> Modular Shield:PINHD-1X8
- JP?: renamed from JP7; value PINHD-1X8BIG -> PINHD-1X8; symbol Raspberry_modular-rescue:PINHD-1X8BIG-OhEye-eagle-import -> Modular Shield:PINHD-1X8
Other:
- note added: "Analog Pin Headers"
- note added: "Analog to Digital Converters"
- note added: "Digital Pin Headers"
- note added: "Mechanicals"
- note added: "Power Flags"
- note added: "Raspberry Pin Headers"
- moved on the sheet: H1, H2, H3, H4, J1, JP1, JP3, JP5, JP?, U$3, U$5, U1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

Commit message: [FIX] Missing annotations
Parts:
- gave numbers to parts that had none: 1
Changed lines of the file:
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@@
   (symbol (lib_id "Modular Shield:PINHD-1X8") (at 203.2 114.3 0) (unit 1)
     (in_bom yes) (on_board yes) (dnp no)
-    (property "Reference" "JP?" (at 196.85 103.505 0)
+    (property "Reference" "JP2" (at 196.85 103.505 0)
       (effects (font (size 1.4986 1.4986)) (justify left bottom))
     )
@@
       (project "Raspberry_modular"
         (path "/f7f606ea-7d0c-4680-9293-4d1bbfd60125"
-          (reference "JP?") (unit 1)
+          (reference "JP2") (unit 1)
         )
       )

Commit message: [UDPT] Electricals footprints
Parts:
- H1, H2, H3, H4: footprint MountingHole:MountingHole_2.7mm_M2.5 -> Modular Shield:MountingHole_2.7mm_M2.5
- J1: footprint Raspberry_modular:PIN_20X2 -> Modular Shield:PIN_20X2
- JP1: value PINHD-1X6B -> PINHD-1X6; footprint Raspberry_modular:1X06-BIG -> Modular Shield:1X06-BIG; symbol Modular Shield:PINHD-1X6B -> Modular Shield:PINHD-1X6
- JP2, JP5: footprint Raspberry_modular:1X08-BIG -> Modular Shield:1X08-BIG
- JP3: value PINHD-1X6B -> PINHD-1X6; footprint Raspberry_modular:1X06-BIG -> Modular Shield:1X06-BIG; symbol Raspberry_modular-rescue:PINHD-1X6B-OhEye-eagle-import -> Modular Shield:PINHD-1X6
- JP4: renamed from U$3; footprint Raspberry_modular:1X10-BIG -> Modular Shield:1X10-BIG
- JP6: renamed from U$5; footprint Raspberry_modular:1X10-BIG -> Modular Shield:1X10-BIG
- R4, R50, R51, R52, R53, R54, R55, R56: footprint Raspberry_modular:R_0603_1608Metric -> Modular Shield:R_0603_1608Metric
- U1, U3: footprint Raspberry_modular:SOIC16 -> Modular Shield:MCP3008 SOIC16
Changed lines of the file:
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@@
   (symbol (lib_id "Modular Shield:PINHD-1X10") (at 172.72 41.91 0) (unit 1)
     (in_bom yes) (on_board yes) (dnp no)
-    (property "Reference" "U$3" (at 166.37 28.575 0)
+    (property "Reference" "JP4" (at 166.37 28.575 0)
       (effects (font (size 1.4986 1.4986)) (justify left bottom))
     )
@@
       (effects (font (size 1.4986 1.4986)) (justify left bottom))
     )
-    (property "Footprint" "Raspberry_modular:1X10-BIG" (at 172.72 41.91 0)
+    (property "Footprint" "Modular Shield:1X10-BIG" (at 172.72 41.91 0)
       (effects (font (size 1.27 1.27)) hide)
     )
@@
       (project "Raspberry_modular"
         (path "/f7f606ea-7d0c-4680-9293-4d1bbfd60125"
-          (reference "U$3") (unit 1)
-        )
-      )
-    )
-  )
-  (symbol (lib_id "Raspberry_modular-rescue:PINHD-1X6B-OhEye-eagle-import") (at 203.2 67.31 0) (unit 1)
+          (reference "JP4") (unit 1)
+        )
+      )
+    )
+  )
+  (symbol (lib_id "Modular Shield:PINHD-1X6") (at 203.2 67.31 0) (unit 1)
     (in_bom yes) (on_board yes) (dnp no)
     (property "Reference" "JP3" (at 196.85 56.515 0)
       (effects (font (size 1.4986 1.4986)) (justify left bottom))
     )
-    (property "Value" "PINHD-1X6B" (at 196.85 77.47 0)
+    (property "Value" "PINHD-1X6" (at 196.85 77.47 0)
       (effects (font (size 1.4986 1.4986)) (justify left bottom))
     )
-    (property "Footprint" "Raspberry_modular:1X06-BIG" (at 203.2 67.31 0)
+    (property "Footprint" "Modular Shield:1X06-BIG" (at 203.2 67.31 0)
       (effects (font (size 1.27 1.27)) hide)
     )
@@
       (effects (font (size 1.27 1.27)) (justify left))
     )
-    (property "Footprint" "MountingHole:MountingHole_2.7mm_M2.5" (at 266.7 110.49 0)
+    (property "Footprint" "Modular Shield:MountingHole_2.7mm_M2.5" (at 266.7 110.49 0)
       (effects (font (size 1.27 1.27)) hide)
     )
@@
       (effects (font (size 1.27 1.27)) (justify left))
     )
-    (property "Footprint" "MountingHole:MountingHole_2.7mm_M2.5" (at 266.7 115.57 0)
+    (property "Footprint" "Modular Shield:MountingHole_2.7mm_M2.5" (at 266.7 115.57 0)
       (effects (font (size 1.27 1.27)) hide)
     )
@@
       (effects (font (size 1.27 1.27)) (justify left))
     )
-    (property "Footprint" "MountingHole:MountingHole_2.7mm_M2.5" (at 266.7 120.65 0)
+    (property "Footprint" "Modular Shield:MountingHole_2.7mm_M2.5" (at 266.7 120.65 0)
       (effects (font (size 1.27 1.27)) hide)
     )
@@
       (effects (font (size 1.27 1.27)) (justify left))
     )
-    (property "Footprint" "MountingHole:MountingHole_2.7mm_M2.5" (at 266.7 125.73 0)
+    (property "Footprint" "Modular Shield:MountingHole_2.7mm_M2.5" (at 266.7 125.73 0)
       (effects (font (size 1.27 1.27)) hide)
     )
@@
       (effects (font (size 1.27 1.27)))
     )
-    (property "Footprint" "Raspberry_modular:R_0603_1608Metric" (at 166.37 179.578 90)
+    (property "Footprint" "Modular Shield:R_0603_1608Metric" (at 166.37 179.578 90)
       (effects (font (size 1.27 1.27)) hide)
     )
@@
       (effects (font (size 1.27 1.27)))
     )
-    (property "Footprint" "Raspberry_modular:R_0603_1608Metric" (at 166.37 184.658 90)
+    (property "Footprint" "Modular Shield:R_0603_1608Metric" (at 166.37 184.658 90)
       (effects (font (size 1.27 1.27)) hide)
     )
@@
       (effects (font (size 1.27 1.27)))
     )
-    (property "Footprint" "Raspberry_modular:R_0603_1608Metric" (at 166.37 189.738 90)
+    (property "Footprint" "Modular Shield:R_0603_1608Metric" (at 166.37 189.738 90)
       (effects (font (size 1.27 1.27)) hide)
     )
@@
       (effects (font (size 1.27 1.27)))
     )
-    (property "Footprint" "Raspberry_modular:R_0603_1608Metric" (at 166.37 194.818 90)
+    (property "Footprint" "Modular Shield:R_0603_1608Metric" (at 166.37 194.818 90)
       (effects (font (size 1.27 1.27)) hide)
     )
@@
       (effects (font (size 1.27 1.27)))
     )
-    (property "Footprint" "Raspberry_modular:R_0603_1608Metric" (at 166.37 199.898 90)
+    (property "Footprint" "Modular Shield:R_0603_1608Metric" (at 166.37 199.898 90)
       (effects (font (size 1.27 1.27)) hide)
     )
@@
       (effects (font (size 1.27 1.27)))
     )
-    (property "Footprint" "Raspberry_modular:R_0603_1608Metric" (at 166.37 204.978 90)
+    (property "Footprint" "Modular Shield:R_0603_1608Metric" (at 166.37 204.978 90)
       (effects (font (size 1.27 1.27)) hide)
     )
@@
       (effects (font (size 1.27 1.27)))
     )
-    (property "Footprint" "Raspberry_modular:R_0603_1608Metric" (at 166.37 210.058 90)
+    (property "Footprint" "Modular Shield:R_0603_1608Metric" (at 166.37 210.058 90)
       (effects (font (size 1.27 1.27)) hide)
     )
@@
       (effects (font (size 1.27 1.27)))
     )
-    (property "Footprint" "Raspberry_modular:SOIC16" (at 275.59 170.18 0)
+    (property "Footprint" "Modular Shield:MCP3008 SOIC16" (at 275.59 170.18 0)
       (effects (font (size 1.27 1.27)) hide)
     )
@@
       (effects (font (size 1.27 1.27)))
     )
-    (property "Footprint" "Raspberry_modular:R_0603_1608Metric" (at 166.37 215.138 90)
+    (property "Footprint" "Modular Shield:R_0603_1608Metric" (at 166.37 215.138 90)
       (effects (font (size 1.27 1.27)) hide)
     )
@@
       (effects (font (size 1.27 1.27)))
     )
-    (property "Footprint" "Raspberry_modular:SOIC16" (at 226.06 170.18 0)
+    (property "Footprint" "Modular Shield:MCP3008 SOIC16" (at 226.06 170.18 0)
       (effects (font (size 1.27 1.27)) hide)
     )
@@
       (effects (font (size 1.27 1.27)))
     )
-    (property "Footprint" "Raspberry_modular:PIN_20X2" (at 69.85 80.01 0)
+    (property "Footprint" "Modular Shield:PIN_20X2" (at 69.85 80.01 0)
       (effects (font (size 1.27 1.27)) hide)
     )
@@
   (symbol (lib_id "Modular Shield:PINHD-1X10") (at 203.2 41.91 0) (unit 1)
     (in_bom yes) (on_board yes) (dnp no)
-    (property "Reference" "U$5" (at 196.85 28.575 0)
+    (property "Reference" "JP6" (at 196.85 28.575 0)
       (effects (font (size 1.4986 1.4986)) (justify left bottom))
     )
@@
       (effects (font (size 1.4986 1.4986)) (justify left bottom))
     )
-    (property "Footprint" "Raspberry_modular:1X10-BIG" (at 203.2 41.91 0)
+    (property "Footprint" "Modular Shield:1X10-BIG" (at 203.2 41.91 0)
       (effects (font (size 1.27 1.27)) hide)
     )
@@
       (project "Raspberry_modular"
         (path "/f7f606ea-7d0c-4680-9293-4d1bbfd60125"
-          (reference "U$5") (unit 1)
-        )
-      )
-    )
-  )
-  (symbol (lib_id "Modular Shield:PINHD-1X6B") (at 172.72 67.31 0) (unit 1)
+          (reference "JP6") (unit 1)
+        )
+      )
+    )
+  )
+  (symbol (lib_id "Modular Shield:PINHD-1X6") (at 172.72 67.31 0) (unit 1)
     (in_bom yes) (on_board yes) (dnp no)
     (property "Reference" "JP1" (at 166.37 56.515 0)
       (effects (font (size 1.4986 1.4986)) (justify left bottom))
     )
-    (property "Value" "PINHD-1X6B" (at 166.37 77.47 0)
+    (property "Value" "PINHD-1X6" (at 166.37 77.47 0)
       (effects (font (size 1.4986 1.4986)) (justify left bottom))
     )
-    (property "Footprint" "Raspberry_modular:1X06-BIG" (at 172.72 67.31 0)
+    (property "Footprint" "Modular Shield:1X06-BIG" (at 172.72 67.31 0)
       (effects (font (size 1.27 1.27)) hide)
     )
@@
       (effects (font (size 1.4986 1.4986)) (justify left bottom))
     )
-    (property "Footprint" "Raspberry_modular:1X08-BIG" (at 172.72 114.3 0)
+    (property "Footprint" "Modular Shield:1X08-BIG" (at 172.72 114.3 0)
       (effects (font (size 1.27 1.27)) hide)
     )
@@
       (effects (font (size 1.4986 1.4986)) (justify left bottom))
     )
-    (property "Footprint" "Raspberry_modular:1X08-BIG" (at 203.2 114.3 0)
-      (effects (font (size 1.27 1.27)) hide)
-    )
+    (property "Footprint" "Modular Shield:1X08-BIG" (at 203.2 114.3 0)
+      (effects (font (size 1.27 1.27)) hide)
+    )

Commit message: [ADD] Bom
Parts:
- H1, H2, H3, H4, J1, JP1, JP2, JP3, JP4, JP5, JP6: now left out of the parts list
- R4, R50, R51, R52, R53, R54, R55, R56: LCSC (none) -> C25804
- U1, U3: LCSC (none) -> C1520159
Other:
- moved on the sheet: JP1, JP3, JP4, JP6
