File: Raspberry_modular_kicad/Raspberry_modular.kicad_pcb (KiCad board)
At the start: 2 copper layers, 65 x 56 mm, 93 parts, among them J1 Raspberry_Pi_2_3, U1 MCP3008, U3 MCP3008

Commit message: [UDPT] Inputs on schematics
Other:
- net class Default removed

Commit message: [UDPT] Electricals footprints
Parts:
- D1, D10, D11, D12, D13, D14, D15, D16, D2, D3, D4, D5, D6, D7, D8, D9: footprint Raspberry_modular:D_0603_1608Metric -> Modular Shield:D_0603_1608Metric
- H1, H2, H3, H4: footprint MountingHole:MountingHole_2.7mm_M2.5 -> Modular Shield:MountingHole_2.7mm_M2.5
- J1: footprint Raspberry_modular:PIN_20X2 -> Modular Shield:PIN_20X2
- JP1, JP3: value PINHD-1X6B -> PINHD-1X6; footprint Raspberry_modular:1X06-BIG -> Modular Shield:1X06-BIG
- JP2: renamed from JP7; value PINHD-1X8BIG -> PINHD-1X8
- JP4: renamed from U$3; footprint Raspberry_modular:1X10-BIG -> Modular Shield:1X10-BIG
- JP5: value PINHD-1X8BIG -> PINHD-1X8; footprint Raspberry_modular:1X08-BIG -> Modular Shield:1X08-BIG
- JP6: renamed from U$5; footprint Raspberry_modular:1X10-BIG -> Modular Shield:1X10-BIG
- R1, R10, R11, R12, R13, R14, R15, R16, R17, R18, R19, R2, R20, R21, R22, R23, R24, R25, R26, R27, R28, R29, R3, R30, R31, R32, R33, R34, R35, R36, R37, R38, R39, R4, R40, R41, R42, R43, R44, R45, R46, R47, R48, R49, R5, R50, R51, R52, R53, R54, R55, R56, R6, R7, R8, R9: footprint Raspberry_modular:R_0603_1608Metric -> Modular Shield:R_0603_1608Metric
- U1, U3: footprint Raspberry_modular:SOIC16 -> Modular Shield:MCP3008 SOIC16
Connections:
- J1 pad 10: (no net) -> unconnected-(J1-GPIO15/RXD-Pad10)
- J1 pad 11: (no net) -> unconnected-(J1-GPIO17-Pad11)
- J1 pad 12: (no net) -> unconnected-(J1-GPIO18/PWM0-Pad12)
- J1 pad 13: (no net) -> unconnected-(J1-GPIO27-Pad13)
- J1 pad 15: (no net) -> unconnected-(J1-GPIO22-Pad15)
- J1 pad 16: (no net) -> unconnected-(J1-GPIO23-Pad16)
- J1 pad 18: (no net) -> unconnected-(J1-GPIO24-Pad18)
- J1 pad 22: (no net) -> unconnected-(J1-GPIO25-Pad22)
- J1 pad 27: (no net) -> unconnected-(J1-ID_SD/GPIO0-Pad27)
- J1 pad 28: (no net) -> unconnected-(J1-ID_SC/GPIO1-Pad28)
- J1 pad 3: (no net) -> unconnected-(J1-SDA/GPIO2-Pad3)
- J1 pad 40: (no net) -> unconnected-(J1-GPIO21/SCLK1-Pad40)
- J1 pad 5: (no net) -> unconnected-(J1-SCL/GPIO3-Pad5)
- J1 pad 7: (no net) -> unconnected-(J1-GCLK0/GPIO4-Pad7)
- J1 pad 8: (no net) -> unconnected-(J1-GPIO14/TXD-Pad8)
Routing:
- net GND: track 154.6 -> 156.1 mm

Commit message: [DRC] Problems fixed
Parts:
- removed the REF** at (58.1, 28.9)
- G***: footprint OhEye:Saturn -> Modular Shield:Saturn
- G***: footprint OhEye:Moon -> Modular Shield:Moon
- G***: footprint OhEye:falling_stars -> Modular Shield:Falling_Stars
- G***: footprint OhEye:cnes -> Modular Shield:CNES
- G***: footprint OhEye:stephen -> Modular Shield:Stephen_Hawking
- G***: footprint OhEye:synth -> Modular Shield:Synthesizer
- REF**: footprint OhEye:ISS -> Modular Shield:ISS
Changed lines of the file:
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@@
     )
   )
-  (footprint "OhEye:ISS" (layer "F.Cu")
+  (footprint "Modular Shield:ISS" (layer "F.Cu")
     (at 75.654 38.824)
     (attr through_hole)
@@
       (stroke (width 0.01) (type solid)) (fill solid) (layer "F.SilkS"))
   )
-  (footprint "OhEye:Saturn" (layer "F.Cu")
+  (footprint "Modular Shield:Saturn" (layer "F.Cu")
     (at 76.924 74.13)
     (attr through_hole)
-    (fp_text reference "G***" (at 0 0) (layer "F.SilkS") hide
+    (fp_text reference "G***" (at -1.1 -5.475) (layer "F.SilkS") hide
         (effects (font (size 1.524 1.524) (thickness 0.3)))
     )
-    (fp_text value "LOGO" (at 0.75 0) (layer "F.SilkS") hide
+    (fp_text value "LOGO" (at -0.525 -11.275) (layer "F.SilkS") hide
         (effects (font (size 1.524 1.524) (thickness 0.3)))
     )
@@
       (stroke (width 0.01) (type solid)) (fill solid) (layer "F.Mask"))
   )
-  (footprint "OhEye:Moon" (layer "F.Cu")
+  (footprint "Modular Shield:Moon" (layer "F.Cu")
     (at 31.458 37.808)
     (attr through_hole)
@@
       (stroke (width 0.01) (type solid)) (fill solid) (layer "F.SilkS"))
   )
-  (footprint "OhEye:falling_stars" (layer "F.Cu")
+  (footprint "Modular Shield:Falling_Stars" (layer "F.Cu")
     (at 57.874 74.13)
     (attr through_hole)
@@
       (stroke (width 0.01) (type solid)) (fill solid) (layer "F.SilkS"))
   )
-  (footprint "OhEye:cnes" (layer "F.Cu")
+  (footprint "Modular Shield:CNES" (layer "F.Cu")
     (at 39.586 76.416)
     (attr through_hole)
-    (fp_text reference "G***" (at 0 0) (layer "F.SilkS") hide
+    (fp_text reference "G***" (at -7.6 -9.4) (layer "F.SilkS") hide
         (effects (font (size 1.524 1.524) (thickness 0.3)))
     )
-    (fp_text value "LOGO" (at 0.75 0) (layer "F.SilkS") hide
+    (fp_text value "LOGO" (at -6.85 -9.4) (layer "F.SilkS") hide
         (effects (font (size 1.524 1.524) (thickness 0.3)))
     )
@@
       (stroke (width 0.01) (type solid)) (fill solid) (layer "F.Mask"))
   )
-  (footprint "OhEye:FemaleBackHeader" (layer "B.Cu")
-    (at 58.128 28.918)
-    (attr through_hole)
-    (fp_text reference "REF**" (at 0 -0.5) (layer "B.SilkS") hide
-        (effects (font (size 1 1) (thickness 0.15)) (justify mirror))
-    )
-    (fp_text value "FemaleBackHeader" (at 0 0.5) (layer "B.Fab")
-        (effects (font (size 1 1) (thickness 0.15)) (justify mirror))
-    )
-    (model "${KISYS3DMOD}/Connector_PinSocket_2.54mm.3dshapes/PinSocket_2x20_P2.54mm_Vertical.step"
-      (offset (xyz 24 -1.4 0))
-      (scale (xyz 1 1 1))
-      (rotate (xyz 0 0 90))
-    )
-  )
-  (footprint "OhEye:stephen" (layer "B.Cu")
+  (footprint "Modular Shield:Stephen_Hawking" (layer "B.Cu")
     (at 60.16 41.872 180)
     (attr through_hole)
@@
       (stroke (width 0.01) (type solid)) (fill solid) (layer "B.SilkS"))
   )
-  (footprint "OhEye:synth" (layer "B.Cu")
+  (footprint "Modular Shield:Synthesizer" (layer "B.Cu")
     (at 57.366 74.13 180)
     (attr through_hole)
