File: Raspberry_modular_kicad/Raspberry_modular.kicad_pcb (KiCad board)
At the start: 2 copper layers, 65 x 56 mm, 92 parts, among them J1 Raspberry_Pi_2_3, U1 MCP3008, U3 MCP3008

Commit message: [ADD] Production build with updated Silk
Other:
- board text added: "6.8V Zener"
- board text removed: "6.6V Zener"
Changed lines of the file:
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@@
     (effects (font (size 0.6 0.6) (thickness 0.1)))
   )
-  (gr_text "6.6V Zener" (at 70.828 48.222) (layer "F.SilkS")
+  (gr_text "6.8V Zener" (at 70.828 48.222) (layer "F.SilkS")
     (effects (font (size 0.6 0.6) (thickness 0.1)))
   )
