File: Modular_Shield_kicad/Modular_Shield.kicad_pcb (KiCad board)
At the start: 2 copper layers, 65 x 56 mm, 92 parts, among them J1 Raspberry_Pi_2_3, U1 MCP3008, U3 MCP3008

Commit message: [UDPT] Kicad Project name
Parts:
- JP2: footprint Raspberry_modular:1X08-BIG -> Modular Shield:1X08-BIG
Changed lines of the file:
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@@
   (footprint "Modular Shield:PIN_20X2" (layer "F.Cu")
     (at 57.956 28.702)
-    (property "Sheetfile" "Raspberry_modular.kicad_sch")
+    (property "Sheetfile" "Modular_Shield.kicad_sch")
     (property "Sheetname" "")
     (property "exclude_from_bom" "")
@@
     (property "JLCPCB Rotation Offset" "270")
     (property "LCSC" "C1520159")
-    (property "Sheetfile" "Raspberry_modular.kicad_sch")
+    (property "Sheetfile" "Modular_Shield.kicad_sch")
     (property "Sheetname" "")
     (property "ki_description" "A/D Converter, 10-Bit, 8-Channel, SPI Interface , 2.7V-5.5V")
@@
     (property "JLCPCB Rotation Offset" "270")
     (property "LCSC" "C1520159")
-    (property "Sheetfile" "Raspberry_modular.kicad_sch")
+    (property "Sheetfile" "Modular_Shield.kicad_sch")
     (property "Sheetname" "")
     (property "ki_description" "A/D Converter, 10-Bit, 8-Channel, SPI Interface , 2.7V-5.5V")
@@
     (descr "Mounting Hole 2.7mm, no annular, M2.5")
     (tags "mounting hole 2.7mm no annular m2.5")
-    (property "Sheetfile" "Raspberry_modular.kicad_sch")
+    (property "Sheetfile" "Modular_Shield.kicad_sch")
     (property "Sheetname" "")
     (property "exclude_from_bom" "")
@@
     (descr "Mounting Hole 2.7mm, no annular, M2.5")
     (tags "mounting hole 2.7mm no annular m2.5")
-    (property "Sheetfile" "Raspberry_modular.kicad_sch")
+    (property "Sheetfile" "Modular_Shield.kicad_sch")
     (property "Sheetname" "")
     (property "exclude_from_bom" "")
@@
     (descr "Mounting Hole 2.7mm, no annular, M2.5")
     (tags "mounting hole 2.7mm no annular m2.5")
-    (property "Sheetfile" "Raspberry_modular.kicad_sch")
+    (property "Sheetfile" "Modular_Shield.kicad_sch")
     (property "Sheetname" "")
     (property "exclude_from_bom" "")
@@
     (descr "Mounting Hole 2.7mm, no annular, M2.5")
     (tags "mounting hole 2.7mm no annular m2.5")
-    (property "Sheetfile" "Raspberry_modular.kicad_sch")
+    (property "Sheetfile" "Modular_Shield.kicad_sch")
     (property "Sheetname" "")
     (property "exclude_from_bom" "")
@@
   (footprint "Modular Shield:1X10-BIG" (layer "F.Cu")
     (at 39.078 66.002)
-    (property "Sheetfile" "Raspberry_modular.kicad_sch")
+    (property "Sheetfile" "Modular_Shield.kicad_sch")
     (property "Sheetname" "")
     (property "exclude_from_bom" "")
@@
       (net 1 "GND") (pinfunction "10") (pintype "passive") (solder_mask_margin 0.0508))
   )
-  (footprint "Raspberry_modular:1X08-BIG" (layer "F.Cu")
+  (footprint "Modular Shield:1X08-BIG" (layer "F.Cu")
     (at 79.21 66.002)
-    (property "Sheetfile" "Raspberry_modular.kicad_sch")
+    (property "Sheetfile" "Modular_Shield.kicad_sch")
     (property "Sheetname" "")
     (property "exclude_from_bom" "")
-    (attr through_hole exclude_from_pos_files exclude_from_bom)
+    (attr through_hole)
     (fp_text reference "JP2" (at -10.2362 -1.8288) (layer "F.SilkS") hide
         (effects (font (size 1.2065 1.2065) (thickness 0.127)) (justify left bottom))
@@
   (footprint "Modular Shield:1X06-BIG" (layer "F.Cu")
     (at 59.398 66.002)
-    (property "Sheetfile" "Raspberry_modular.kicad_sch")
+    (property "Sheetfile" "Modular_Shield.kicad_sch")
     (property "Sheetname" "")
     (property "exclude_from_bom" "")
@@
   (footprint "Modular Shield:1X10-BIG" (layer "F.Cu")
     (at 39.078 63.462)
-    (property "Sheetfile" "Raspberry_modular.kicad_sch")
+    (property "Sheetfile" "Modular_Shield.kicad_sch")
     (property "Sheetname" "")
     (property "exclude_from_bom" "")
@@
   (footprint "Modular Shield:1X08-BIG" (layer "F.Cu")
     (at 79.21 63.462)
-    (property "Sheetfile" "Raspberry_modular.kicad_sch")
+    (property "Sheetfile" "Modular_Shield.kicad_sch")
     (property "Sheetname" "")
     (property "exclude_from_bom" "")
@@
   (footprint "Modular Shield:1X06-BIG" (layer "F.Cu")
     (at 59.398 63.462)
-    (property "Sheetfile" "Raspberry_modular.kicad_sch")
+    (property "Sheetfile" "Modular_Shield.kicad_sch")
     (property "Sheetname" "")
     (property "exclude_from_bom" "")
@@
     (tags "resistor")
     (property "LCSC" "C25804")
-    (property "Sheetfile" "Raspberry_modular.kicad_sch")
+    (property "Sheetfile" "Modular_Shield.kicad_sch")
     (property "Sheetname" "")
     (property "ki_description" "Resistor")
@@
     (tags "resistor")
     (property "LCSC" "C25804")
-    (property "Sheetfile" "Raspberry_modular.kicad_sch")
+    (property "Sheetfile" "Modular_Shield.kicad_sch")
     (property "Sheetname" "")
     (property "ki_description" "Resistor")
@@
     (tags "resistor")
     (property "LCSC" "C25804")
-    (property "Sheetfile" "Raspberry_modular.kicad_sch")
+    (property "Sheetfile" "Modular_Shield.kicad_sch")
     (property "Sheetname" "")
     (property "ki_description" "Resistor")
@@
     (tags "resistor")
     (property "LCSC" "C25804")
-    (property "Sheetfile" "Raspberry_modular.kicad_sch")
+    (property "Sheetfile" "Modular_Shield.kicad_sch")
     (property "Sheetname" "")
     (property "ki_description" "Resistor")
@@
     (tags "resistor")
     (property "LCSC" "C25804")
-    (property "Sheetfile" "Raspberry_modular.kicad_sch")
+    (property "Sheetfile" "Modular_Shield.kicad_sch")
     (property "Sheetname" "")
     (property "ki_description" "Resistor")
@@
     (tags "resistor")
     (property "LCSC" "C25804")
-    (property "Sheetfile" "Raspberry_modular.kicad_sch")
+    (property "Sheetfile" "Modular_Shield.kicad_sch")
     (property "Sheetname" "")
     (property "ki_description" "Resistor")
@@
     (tags "resistor")
     (property "LCSC" "C25804")
-    (property "Sheetfile" "Raspberry_modular.kicad_sch")
+    (property "Sheetfile" "Modular_Shield.kicad_sch")
     (property "Sheetname" "")
     (property "ki_description" "Resistor")
@@
     (tags "resistor")
     (property "LCSC" "C25804")
-    (property "Sheetfile" "Raspberry_modular.kicad_sch")
+    (property "Sheetfile" "Modular_Shield.kicad_sch")
     (property "Sheetname" "")
     (property "ki_description" "Resistor")
