File: Modular_Shield_kicad/Modular_Shield.kicad_pcb (KiCad board)
At the start: 2 copper layers, 65 x 56 mm, 92 parts, among them J1 Raspberry_Pi_2_3, U1 MCP3008, U3 MCP3008

Commit message: [FIX] Missing Text On IBOM
Other:
- board text removed: "juthomas.fr"
Changed lines of the file:
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@@
         (effects (font (size 1.524 1.524) (thickness 0.3)))
     )
+    (fp_text user "juthomas.fr" (at 0 4.572 unlocked) (layer "F.Cu")
+        (effects (font (size 1.6 1.6) (thickness 0.25)))
+    )
     (fp_text user "G***" (at -1.1 -5.475) (layer "F.SilkS") hide
         (effects (font (size 1.524 1.524) (thickness 0.3)))
     )
+    (fp_text user "juthomas.fr" (at 0 4.572 unlocked) (layer "F.Mask")
+        (effects (font (size 1.6 1.6) (thickness 0.25)))
+    )
     (fp_poly
       (pts
@@
   (gr_line (start 86.956 81.202) (end 28.956 81.202)
     (stroke (width 0.05) (type solid)) (layer "Edge.Cuts"))
-  (gr_text "juthomas.fr" (at 76.162 78.956) (layer "F.Cu")
-    (effects (font (size 1.6 1.6) (thickness 0.25)))
-  )
   (gr_text "So long as the universe had a beginning, \nwe could suppose it had a creator. \nBut if the universe is really completely self-contained, \nhaving no boundary or edge, \nit would have neither beginning nor end: \nit would simply be. What place, then, for a creator?" (at 76.924 56.858) (layer "B.SilkS")
     (effects (font (size 1 1) (thickness 0.15)) (justify left mirror))
@@
     (effects (font (size 0.6 0.6) (thickness 0.1)))
   )
-  (gr_text "juthomas.fr" (at 76.162 78.956) (layer "F.Mask")
-    (effects (font (size 1.6 1.6) (thickness 0.25)))
-  )
   (segment (start 30.188 50.89) (end 30.94041 50.13759) (width 0.25) (layer "F.Cu") (net 1))
